Commit message: add controller and examples

File: KinovaPy/assets/urdf/GEN3-7DOF-VISION_ARM_URDF_V12.urdf (robot description, URDF)
Before this commit: robot GEN3-7DOF-VISION_ARM_URDF_V12, 12 links, 11 joints
Joints:
- joint joint_1: limit effort=39 velocity=1.3963 -> lower=-1.57 upper=1.57 effort=39 velocity=1.3963
- joint joint_2: limit lower=-2.24 upper=2.24 effort=39 velocity=1.3963 -> lower=-0.79 upper=1.57 effort=39 velocity=1.3963
- joint joint_3: limit effort=39 velocity=1.3963 -> lower=-6.28 upper=6.28 effort=39 velocity=1.3963
- joint joint_5: limit effort=9 velocity=1.2218 -> lower=-6.28 upper=6.28 effort=9 velocity=1.2218
- joint joint_7: limit effort=9 velocity=1.2218 -> lower=-6.28 upper=6.28 effort=9 velocity=1.2218
